Commit message: added xacro partial template

File: rover_description/urdf/core.xacro (robot description, xacro)
@@ -8,4 +8,6 @@
           <box size="${size}"/>
         </geometry>
+        <material name="${body_colour}"/>
+        <xacro:gaz_colour name="${name}" colour="${body_colour}"/>
       </visual>
     </link>
@@ -24,4 +26,6 @@
           <cylinder radius="${wheel_radius}" length="${wheel_length}"/>
         </geomentry>
+        <material name="${wheel_colour}"/>
+        <xacro:gaz_colour name="${name}" colour="${wheel_colour}"/>
       </visual>
     </link>

File: rover_description/urdf/gazebo.xacro (robot description, xacro)
@@ -0,0 +1,7 @@
+<robot name="rover">
+  <!--gazebo parameters-->
+  <!--gazebo visuals-->
+  <xacro:include filename="$(find rover_description)/urdf/gazebo_visuals.xacro"/>
+  <!--gazebo physics-->
+  <xacro:include filename="$(find rover_description)/urdf/gazebo_physics.xacro"/>
+</robot>
